File: pcb/traffic_light.kicad_pcb (KiCad board)
At the start: 2 copper layers, 35 x 130 mm, 54 parts, among them Q1 BS170, Q2 BS170, Q3 BS170, SW1 Power_Switch, U1 ESP-12F, U2 AMS1117-3.3

Commit message: Minor PCB improvements
Parts:
- removed SW1: Power_Switch, Connector_PinHeader_2.54mm:PinHeader_1x02_P2.54mm_Vertical
Connections:
- UART1 pad 1: VCC -> +5V
- VIN1 pad 2: Net-(SW1-Pad1) -> +5V
Routing:
- net VCC: track 129.0 -> 113.3 mm
- net +5V: track 134.7 -> 139.3 mm
- net Net-(SW1-Pad1): track 4.63 -> 0.00 mm
Other:
- board text added: "+5V"
- board text added: "Traffic Light v1.1 Ilya Strukov"
- board text removed: "+3.3V"
- board text removed: "Traffic Light v1 Ilya Strukov"
Changed lines of the file:
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@@
-(kicad_pcb (version 20171130) (host pcbnew "(5.0.1-3-g963ef8bb5)")
+(kicad_pcb (version 20171130) (host pcbnew "(5.1.0-0)")
   (general
     (thickness 1.6)
     (drawings 11)
-    (tracks 214)
+    (tracks 213)
     (zones 0)
-    (modules 54)
-    (nets 33)
+    (modules 53)
+    (nets 32)
   )
   (page A4)
@@
     (zone_45_only no)
     (trace_min 0.2)
-    (segment_width 0.2)
-    (edge_width 0.15)
     (via_size 0.8)
     (via_drill 0.4)
@@
     (uvia_min_size 0.2)
     (uvia_min_drill 0.1)
+    (edge_width 0.15)
+    (segment_width 0.2)
     (pcb_text_width 0.3)
     (pcb_text_size 1.5 1.5)
@@
   (net 30 "Net-(U1-Pad15)")
   (net 31 "Net-(U1-Pad16)")
-  (net 32 "Net-(SW1-Pad1)")
   (net_class Default "This is the default net class."
     (clearance 0.2)
@@
     (add_net "Net-(R22-Pad1)")
     (add_net "Net-(R23-Pad2)")
-    (add_net "Net-(SW1-Pad1)")
     (add_net "Net-(U1-Pad15)")
     (add_net "Net-(U1-Pad16)")
@@
   )
   (module Connector_PinHeader_2.54mm:PinHeader_1x02_P2.54mm_Vertical (layer F.Cu)
-    (at 51.85 150)
-    (descr "Through hole straight pin header, 1x02, 2.54mm pitch, single row")
-    (tags "Through hole pin header THT 1x02 2.54mm single row")
-    (fp_text reference SW1 (at 2.5 1.3 90) (layer F.SilkS)
-      (effects (font (size 1 1) (thickness 0.15)))
-    )
-    (fp_text value Power_Switch (at 0 4.87) (layer F.Fab)
-      (effects (font (size 1 1) (thickness 0.15)))
-    )
-    (fp_text user %R (at 0 1.27 90) (layer F.Fab)
-      (effects (font (size 1 1) (thickness 0.15)))
-    )
-    (fp_line (start 1.8 -1.8) (end -1.8 -1.8) (layer F.CrtYd) (width 0.05))
-    (fp_line (start 1.8 4.35) (end 1.8 -1.8) (layer F.CrtYd) (width 0.05))
-    (fp_line (start -1.8 4.35) (end 1.8 4.35) (layer F.CrtYd) (width 0.05))
-    (fp_line (start -1.8 -1.8) (end -1.8 4.35) (layer F.CrtYd) (width 0.05))
-    (fp_line (start -1.33 -1.33) (end 0 -1.33) (layer F.SilkS) (width 0.12))
-    (fp_line (start -1.33 0) (end -1.33 -1.33) (layer F.SilkS) (width 0.12))
-    (fp_line (start -1.33 1.27) (end 1.33 1.27) (layer F.SilkS) (width 0.12))
-    (fp_line (start 1.33 1.27) (end 1.33 3.87) (layer F.SilkS) (width 0.12))
-    (fp_line (start -1.33 1.27) (end -1.33 3.87) (layer F.SilkS) (width 0.12))
-    (fp_line (start -1.33 3.87) (end 1.33 3.87) (layer F.SilkS) (width 0.12))
-    (fp_line (start -1.27 -0.635) (end -0.635 -1.27) (layer F.Fab) (width 0.1))
-    (fp_line (start -1.27 3.81) (end -1.27 -0.635) (layer F.Fab) (width 0.1))
-    (fp_line (start 1.27 3.81) (end -1.27 3.81) (layer F.Fab) (width 0.1))
-    (fp_line (start 1.27 -1.27) (end 1.27 3.81) (layer F.Fab) (width 0.1))
-    (fp_line (start -0.635 -1.27) (end 1.27 -1.27) (layer F.Fab) (width 0.1))
-    (pad 2 thru_hole oval (at 0 2.54) (size 1.7 1.7) (drill 1) (layers *.Cu *.Mask)
-      (net 21 +5V))
-    (pad 1 thru_hole rect (at 0 0) (size 1.7 1.7) (drill 1) (layers *.Cu *.Mask)
-      (net 32 "Net-(SW1-Pad1)"))
-    (model ${KISYS3DMOD}/Connector_PinHeader_2.54mm.3dshapes/PinHeader_1x02_P2.54mm_Vertical.wrl
-      (at (xyz 0 0 0))
-      (scale (xyz 1 1 1))
-      (rotate (xyz 0 0 0))
-    )
-  )
-  (module Connector_PinHeader_2.54mm:PinHeader_1x02_P2.54mm_Vertical (layer F.Cu)
     (at 51.8 142.85)
     (descr "Through hole straight pin header, 1x02, 2.54mm pitch, single row")
     (tags "Through hole pin header THT 1x02 2.54mm single row")
-    (fp_text reference VIN1 (at 2.25 1.45 90) (layer F.SilkS)
+    (fp_text reference VIN1 (at 0.2 -2.55 180) (layer F.SilkS)
       (effects (font (size 1 1) (thickness 0.15)))
     )
@@
       (net 2 GND))
     (pad 2 thru_hole oval (at 0 2.54) (size 1.7 1.7) (drill 1) (layers *.Cu *.Mask)
-      (net 32 "Net-(SW1-Pad1)"))
+      (net 21 +5V))
     (model ${KISYS3DMOD}/Connector_PinHeader_2.54mm.3dshapes/PinHeader_1x02_P2.54mm_Vertical.wrl
       (at (xyz 0 0 0))
@@
     )
     (pad 1 thru_hole rect (at 0 0) (size 1.7 1.7) (drill 1) (layers *.Cu *.Mask)
-      (net 1 VCC))
+      (net 21 +5V))
     (pad 2 thru_hole oval (at 0 2.54) (size 1.7 1.7) (drill 1) (layers *.Cu *.Mask)
       (net 2 GND))
@@
     )
   )
-  (gr_text +3.3V (at 55.35 70.8) (layer F.SilkS)
+  (gr_text +5V (at 55.35 70.8) (layer F.SilkS)
     (effects (font (size 1 1) (thickness 0.15)))
   )
@@
     (effects (font (size 1 1) (thickness 0.15)))
   )
-  (gr_text "Traffic Light v1\nIlya Strukov" (at 73.95 146.65) (layer F.SilkS)
+  (gr_text "Traffic Light v1.1\nIlya Strukov" (at 73.95 146.65) (layer F.SilkS)
     (effects (font (size 1.5 1.5) (thickness 0.3)))
   )
@@
   (segment (start 66.3 73.8) (end 63.7625 76.3375) (width 0.5) (layer F.Cu) (net 1))
   (segment (start 67.147998 73.8) (end 66.3 73.8) (width 0.5) (layer F.Cu) (net 1))
-  (segment (start 63.3 70.8) (end 51.9 70.8) (width 0.5) (layer F.Cu) (net 1))
-  (segment (start 66.3 73.8) (end 63.3 70.8) (width 0.5) (layer F.Cu) (net 1))
   (via (at 66.2 91.55) (size 0.8) (drill 0.4) (layers F.Cu B.Cu) (net 2))
   (via (at 72.8 81.65) (size 0.8) (drill 0.4) (layers F.Cu B.Cu) (net 2))
@@
   (segment (start 52.5125 108.5875) (end 54 107.1) (width 0.5) (layer F.Cu) (net 21))
   (segment (start 52.5125 109.5) (end 52.5125 108.5875) (width 0.5) (layer F.Cu) (net 21))
-  (segment (start 52.6625 66.5) (end 55.2125 69.05) (width 0.5) (layer F.Cu) (net 21))
-  (segment (start 55.2125 69.05) (end 55.3 69.05) (width 0.5) (layer F.Cu) (net 21))
-  (via (at 55.3 69.05) (size 0.8) (drill 0.4) (layers F.Cu B.Cu) (net 21))
-  (segment (start 59 72.75) (end 55.3 69.05) (width 0.5) (layer B.Cu) (net 21))
-  (segment (start 59 102.1) (end 59 72.75) (width 0.5) (layer B.Cu) (net 21))
-  (segment (start 54 107.1) (end 59 102.1) (width 0.5) (layer B.Cu) (net 21))
   (segment (start 56.95 149.5) (end 57.1 149.65) (width 0.5) (layer F.Cu) (net 21))
   (segment (start 56.95 147.05) (end 56.95 149.5) (width 0.5) (layer F.Cu) (net 21))
-  (segment (start 51.85 161.0875) (end 52.5125 161.75) (width 0.5) (layer F.Cu) (net 21))
-  (segment (start 51.85 152.54) (end 51.85 161.0875) (width 0.5) (layer F.Cu) (net 21))
-  (segment (start 54.35 139.9) (end 52.5125 138.0625) (width 0.5) (layer F.Cu) (net 21))
-  (segment (start 52.5125 138.0625) (end 52.5125 122.5) (width 0.5) (layer F.Cu) (net 21))
-  (segment (start 53.052081 152.54) (end 54.35 151.242081) (width 0.5) (layer F.Cu) (net 21))
-  (segment (start 51.85 152.54) (end 53.052081 152.54) (width 0.5) (layer F.Cu) (net 21))
-  (segment (start 56.95 147.05) (end 55.975 147.05) (width 0.5) (layer F.Cu) (net 21))
-  (segment (start 54.35 147.05) (end 54.35 139.9) (width 0.5) (layer F.Cu) (net 21))
-  (segment (start 55.975 147.05) (end 54.35 147.05) (width 0.5) (layer F.Cu) (net 21))
-  (segment (start 54.35 151.242081) (end 54.35 147.05) (width 0.5) (layer F.Cu) (net 21))
+  (segment (start 52.5125 161.75) (end 51.8 161.0375) (width 0.5) (layer F.Cu) (net 21))
+  (segment (start 51.85 147.05) (end 51.8 147) (width 0.5) (layer F.Cu) (net 21))
+  (segment (start 56.95 147.05) (end 51.85 147.05) (width 0.5) (layer F.Cu) (net 21))
+  (segment (start 51.8 147) (end 51.8 145.39) (width 0.5) (layer F.Cu) (net 21))
+  (segment (start 51.8 161.0375) (end 51.8 147) (width 0.5) (layer F.Cu) (net 21))
+  (via (at 55.4 70.700002) (size 0.8) (drill 0.4) (layers F.Cu B.Cu) (net 21))
+  (segment (start 51.999998 70.700002) (end 51.9 70.8) (width 0.5) (layer F.Cu) (net 21))
+  (segment (start 55.4 70.700002) (end 51.999998 70.700002) (width 0.5) (layer F.Cu) (net 21))
+  (segment (start 52.6625 70.0375) (end 51.9 70.8) (width 0.5) (layer F.Cu) (net 21))
+  (segment (start 52.6625 66.5) (end 52.6625 70.0375) (width 0.5) (layer F.Cu) (net 21))
+  (segment (start 55.500002 70.700002) (end 55.4 70.700002) (width 0.5) (layer B.Cu) (net 21))
+  (segment (start 59.6 74.8) (end 55.500002 70.700002) (width 0.5) (layer B.Cu) (net 21))
+  (segment (start 59.6 101.5) (end 59.6 74.8) (width 0.5) (layer B.Cu) (net 21))
+  (segment (start 54 107.1) (end 59.6 101.5) (width 0.5) (layer B.Cu) (net 21))
+  (segment (start 53.283847 123.271347) (end 52.5125 122.5) (width 0.5) (layer F.Cu) (net 21))
+  (segment (start 53.4 123.3875) (end 53.283847 123.271347) (width 0.5) (layer F.Cu) (net 21))
+  (segment (start 53.4 144.120002) (end 53.4 123.3875) (width 0.5) (layer F.Cu) (net 21))
+  (segment (start 52.130002 145.39) (end 53.4 144.120002) (width 0.5) (layer F.Cu) (net 21))
+  (segment (start 51.8 145.39) (end 52.130002 145.39) (width 0.5) (layer F.Cu) (net 21))
   (segment (start 80.683847 66.228653) (end 79.9125 67) (width 0.25) (layer F.Cu) (net 22))
   (segment (start 82.275001 58.805001) (end 82.275001 64.637499) (width 0.25) (layer F.Cu) (net 22))
@@
   (segment (start 55.47 78.42) (end 51.9 78.42) (width 0.25) (layer F.Cu) (net 31))
   (segment (start 58.8 81.75) (end 55.47 78.42) (width 0.25) (layer F.Cu) (net 31))
-  (segment (start 51.85 145.44) (end 51.8 145.39) (width 0.25) (layer F.Cu) (net 32))
-  (segment (start 51.85 150) (end 51.85 145.44) (width 0.25) (layer F.Cu) (net 32))
   (zone (net 2) (net_name GND) (layer F.Cu) (hatch edge 0.508)
     (connect_pads (clearance 0.508))
